File: Lighting board/_saved_Lighting board.sch (KiCad schematic (older format))
At the start: 16 parts, among them SW1 SW_SPDT, U1 LDD-1500L, U2 LDD-1500L, U3 TM4C129E_Launchpad, U4 OKI

Commit message: Schematic/High Level Block Diagram
Parts:
- Conn1C1, Conn1D1: footprint MRDT_Connectors:MOLEX_SL_02_Vertical -> MRDT_Connectors:MOLEX_SL_02_Horizontal
Changed lines of the file:
@@
 F 0 "Conn1C1" H 3377 4508 60  0000 L CNN
 F 1 "Molex_SL_02" H 3377 4402 60  0000 L CNN
-F 2 "MRDT_Connectors:MOLEX_SL_02_Vertical" H 3250 4250 60  0001 C CNN
+F 2 "MRDT_Connectors:MOLEX_SL_02_Horizontal" H 3250 4250 60  0001 C CNN
 F 3 "" H 3250 4250 60  0001 C CNN
 	1    3250 4350
@@
 F 0 "Conn1D1" H 3377 5458 60  0000 L CNN
 F 1 "Molex_SL_02" H 3377 5352 60  0000 L CNN
-F 2 "MRDT_Connectors:MOLEX_SL_02_Vertical" H 3250 5200 60  0001 C CNN
+F 2 "MRDT_Connectors:MOLEX_SL_02_Horizontal" H 3250 5200 60  0001 C CNN
 F 3 "" H 3250 5200 60  0001 C CNN
 	1    3250 5300
