File: LightingBoard_Hardware/LightingBoard_Hardware.kicad_pcb (KiCad board)
At the start: 2 copper layers, 61 x 108.2 mm, 20 parts, among them U1 LDD-1500L, U2 LDD-1500L, U3 TM4C129E_Launchpad, U4 AP1059

Commit message: Fixed Scematic for the nth time
Parts:
- removed C1, C2, C3: 10uF, Capacitor_SMD:C_0603_1608Metric_Pad1.05x0.95mm_HandSolder
- removed Conn1: AndersonPP, MRDT_Connectors:Anderson_3_Horisontal_Side_by_Side
- removed Conn1C1, Conn1D1: Molex_SL_02, MRDT_Connectors:MOLEX_SL_02_Horizontal
- removed Conn2C1: Molex_SL_03, MRDT_Connectors:MOLEX_SL_03_Horizontal
- removed D1: D_Schottky, Diode_SMD:D_0603_1608Metric_Pad1.05x0.95mm_HandSolder
- removed D2: G_LED, LED_SMD:LED_0603_1608Metric_Pad1.05x0.95mm_HandSolder
- removed D3, D4: Org_LED, LED_SMD:LED_0603_1608Metric_Pad1.05x0.95mm_HandSolder
- removed L1: 47uH, Inductor_SMD:L_0603_1608Metric_Pad1.05x0.95mm_HandSolder
- removed R1: 470, Resistor_SMD:R_0603_1608Metric_Pad1.05x0.95mm_HandSolder
- removed R2, R3, R4: 500, Resistor_SMD:R_0603_1608Metric_Pad1.05x0.95mm_HandSolder
- removed U1, U2: LDD-1500L, Project Library:LDD-1500L_LED_DRIVER
- removed U3: TM4C129E_Launchpad, MRDT_Shields:TM4C129E_Launchpad_X9_Bottom_SMD
- removed U4: AP1059, Package_SO:SO-8_5.3x6.2mm_P1.27mm
Routing:
- net +5V: track 141.0 -> 0.00 mm, vias 1 -> 0
- net Dout_NeoPixel: track 104.4 -> 0.00 mm
- net /Headlight_V2-: track 85.0 -> 0.00 mm
- net Headlight_OnOff_PWM1: track 76.9 -> 0.00 mm
- net /Headlight_V1-: track 56.7 -> 0.00 mm
- net /Headlight_V2+: track 55.3 -> 0.00 mm
- net /+12V: track 47.1 -> 0.00 mm
- net +12VA: track 36.6 -> 0.00 mm
- net /Headlight_V1+: track 29.1 -> 0.00 mm
- net GND: track 24.0 -> 0.00 mm, vias 2 -> 0
- net Headlight_OnOff_PWM2: track 16.3 -> 0.00 mm
- net Net-(D1-Pad1): track 7.58 -> 0.00 mm
- net Net-(Conn2C1-Pad2): track 3.90 -> 0.00 mm
- net Net-(U2-Pad1): track 2.54 -> 0.00 mm
- net Net-(D4-Pad2): track 2.06 -> 0.00 mm
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- removed copper zone on B.Cu, net GND
- removed copper zone on F.Cu, net GND
Other:
- board outline removed
- board text removed: "LED Drivers"
- board text removed: "Lighting Hardware, Rev 1 Mars Rover Design Team Missouri S&T, 2019 Name1, Name 2"
- board text removed: "Neo_Pixel_Strip"
- board text removed: "Power"
- board text removed: "Power_In"
- board text removed: "Software"

Commit message: PCB Layout Finished
Parts:
- added C1: 10uF, Capacitor_SMD:C_0603_1608Metric_Pad1.05x0.95mm_HandSolder, F.Cu at (118.9, 50.4)
- added C2: 10uF, Capacitor_SMD:C_0603_1608Metric_Pad1.05x0.95mm_HandSolder, F.Cu at (139.2, 123.3)
- added C3: 10uF, Capacitor_SMD:C_0603_1608Metric_Pad1.05x0.95mm_HandSolder, F.Cu at (132.3, 123.3)
- added Conn1: AndersonPP, MRDT_Connectors:Anderson_3_Horisontal_Side_by_Side, F.Cu at (116.7, 116.5)
- added Conn2: Molex_SL_02, MRDT_Connectors:MOLEX_SL_02_Horizontal, F.Cu at (115.3, 68.2)
- added Conn3: Molex_SL_02, MRDT_Connectors:MOLEX_SL_02_Horizontal, F.Cu at (115.3, 58.7)
- added Conn4: Molex_SL_03, MRDT_Connectors:MOLEX_SL_03_Horizontal, F.Cu at (115.3, 47.9)
- added D2: G_LED, LED_SMD:LED_0603_1608Metric_Pad1.05x0.95mm_HandSolder, F.Cu at (142.5, 43.6)
- added D3: Org_LED, LED_SMD:LED_0603_1608Metric_Pad1.05x0.95mm_HandSolder, F.Cu at (151.0, 43.6)
- added D4: Org_LED, LED_SMD:LED_0603_1608Metric_Pad1.05x0.95mm_HandSolder, F.Cu at (159.5, 43.6)
- added R1: 470, Resistor_SMD:R_0603_1608Metric_Pad1.05x0.95mm_HandSolder, F.Cu at (118.9, 47.9)
- added R2: 500, Resistor_SMD:R_0603_1608Metric_Pad1.05x0.95mm_HandSolder, F.Cu at (138.5, 43.6)
- added R3: 500, Resistor_SMD:R_0603_1608Metric_Pad1.05x0.95mm_HandSolder, F.Cu at (147.1, 43.6)
- added R4: 500, Resistor_SMD:R_0603_1608Metric_Pad1.05x0.95mm_HandSolder, F.Cu at (155.6, 43.6)
- added U1: LDD-1500L, MRDT_Devices:LDD-1500L_LED_DRIVER, F.Cu at (160.5, 101.2)
- added U2: LDD-1500L, MRDT_Devices:LDD-1500L_LED_DRIVER, F.Cu at (160.5, 79.6)
- added U3: TM4C129E_Launchpad, MRDT_Shields:TM4C129E_Launchpad_X9_SMD, F.Cu at (101.5, 123.6)
- added U4: OKI, MRDT_Devices:OKI_Horizontal, F.Cu at (140.8, 120.9)
Routing:
- net +5V: track 0.00 -> 7.75 mm, vias 0 -> 1
- net Net-(C2-Pad1): track 0.00 -> 3.68 mm
- net Net-(Conn4-Pad2): track 0.00 -> 2.67 mm
- net Net-(D2-Pad2): track 0.00 -> 2.22 mm
- net Net-(D4-Pad2): track 0.00 -> 2.16 mm
- net Net-(D3-Pad2): track 0.00 -> 2.16 mm
- net GND: track 0.00 -> 1.65 mm, vias 0 -> 1
- added copper zone on B.Cu, net +5V
- added copper zone on F.Cu, net GND
Other:
- board outline added: 61 x 108.8 mm
- board text added: "HL"
- board text added: "HL1"
- board text added: "HL2"
- board text added: "NeoP"
- board text added: "NeoPixel"
- board text added: "Power"

Commit message: Traces are finished
Parts:
- added ?: , , F.Cu at (134.6, 121.8)
- U4: value OKI -> +5V OKI
- moved U1 37.7 mm to (128.8, 80.9), turned to 270 degrees
- moved U2 37.7 mm to (128.8, 59.3), turned to 270 degrees
Connections:
- Conn1 pad 2: Net-(C2-Pad1) -> +12VA
- Conn1 pad 3: +12VA -> Net-(C2-Pad1)
Routing:
- net Headlight_OnOff_PWM1: track 0.00 -> 111.4 mm
- net Dout_NeoPixel: track 0.00 -> 77.7 mm, vias 0 -> 1
- net +12VA: track 0.00 -> 67.0 mm
- net /Headlight_V1+: track 0.00 -> 43.5 mm
- net Headlight_OnOff_PWM2: track 0.00 -> 38.6 mm
- net /Headlight_V1-: track 0.00 -> 31.9 mm
- net /Headlight_V2+: track 0.00 -> 31.5 mm
- net Net-(C2-Pad1): track 3.68 -> 27.1 mm
- net /Headlight_V2-: track 0.00 -> 19.9 mm
- net GND: track 1.65 -> 8.38 mm, vias 1 -> 2
Other:
- board text added: "+"
