File: LightingBoard_Hardware/LightingBoard_Hardware.sch (KiCad schematic (older format))
At the start: 24 parts, among them SW1 SW_Push, SW2 SW_Push, SW3 SW_Push, U1 LDD-1500L, U2 LDD-1500L, U3 TM4C129E_Launchpad, U4 OKI

Commit message: Added push buttons
cleaned up
Connections:
- net Headlight_Power: now also U3.PM3 (D1_2); no longer U3.PA6 (B1_8)
- net NeoPixel_Pattern: now also U3.PL5 (C1_6); no longer U3.PM5 (B1_10)
- net NeoPixel_White: now also U3.PL4 (C1_5); no longer U3.PM4 (B1_9)
Changed lines of the file:
@@
 L power:GND #PWR0103
 U 1 1 5C05151B
-P 4700 1300
-F 0 "#PWR0103" H 4700 1050 50  0001 C CNN
-F 1 "GND" H 4705 1127 50  0000 C CNN
-F 2 "" H 4700 1300 50  0001 C CNN
-F 3 "" H 4700 1300 50  0001 C CNN
-	1    4700 1300
+P 4000 1300
+F 0 "#PWR0103" H 4000 1050 50  0001 C CNN
+F 1 "GND" H 4005 1127 50  0000 C CNN
+F 2 "" H 4000 1300 50  0001 C CNN
+F 3 "" H 4000 1300 50  0001 C CNN
+	1    4000 1300
 	1    0    0    -1
 $EndComp
@@
 	5850 1300 5900 1300
 Wire Wire Line
-	4850 1300 4700 1300
-Wire Wire Line
 	4800 1800 4850 1800
 Wire Wire Line
@@
 Wire Notes Line
 	475  5075 10325 5075
-Text GLabel 6725 2000 0    50   Input ~ 0
+Text GLabel 4800 1400 0    50   Input ~ 0
 Headlight_Power
-Text GLabel 6725 2100 0    50   Input ~ 0
+Text GLabel 5900 1700 2    50   Input ~ 0
 NeoPixel_White
-Text GLabel 6725 2200 0    50   Input ~ 0
+Text GLabel 5900 1800 2    50   Input ~ 0
 NeoPixel_Pattern
 Wire Wire Line
-	6725 2000 6800 2000
-Wire Wire Line
-	6725 2100 6800 2100
-Wire Wire Line
-	6725 2200 6800 2200
+	5850 1700 5900 1700
+Wire Wire Line
+	5850 1800 5900 1800
+Wire Wire Line
+	4850 1400 4800 1400
+Wire Wire Line
+	4000 1300 4850 1300
 $EndSCHEMATC
