File: LightingBoard_Hardware/LightingBoard_Hardware.sch (KiCad schematic (older format))
At the start: 20 parts, among them U1 LDD-1500L, U2 LDD-1500L, U3 TM4C129E_Launchpad, U4 AP1059

Commit message: Fixed Schematic
Parts:
- removed C2, C3: 10uF, Capacitor_SMD:C_0603_1608Metric_Pad1.05x0.95mm_HandSolder, symbol Device:C
- removed D1: D_Schottky, Diode_SMD:D_0603_1608Metric_Pad1.05x0.95mm_HandSolder, symbol Device:D_Schottky
- removed L1: 47uH, LightingBoard_Hardware2:ETQ-P4M470YFN_Inductor, symbol pspice:INDUCTOR
- removed U4: AP1059, Package_SO:SO-8_5.3x6.2mm_P1.27mm, symbol MRDT_ICs:AP1059
- added C? (x2): 10uF, Capacitor_SMD:C_0603_1608Metric_Pad1.05x0.95mm_HandSolder, symbol Device:C_Small
- added U?: OKI, symbol MRDT_Devices:OKI
Connections:
- net labels removed: +12V
- wire segments 80 -> 71
Changed lines of the file:
@@
 EESchema Schematic File Version 4
+LIBS:LightingBoard_Hardware-cache
 EELAYER 26 0
 EELAYER END
@@
 Text Label 2450 3550 0    50   ~ 0
 Headlight_V1+
-Text Label 1950 1400 0    50   ~ 0
-+12V
 Wire Wire Line
 	1450 3400 1450 3450
@@
 	0    1    1    0
 $EndComp
-$Comp
-L Device:C C2
-U 1 1 5BDE3ABA
-P 1800 1650
-F 0 "C2" H 1550 1650 50  0000 L CNN
-F 1 "10uF" H 1500 1750 50  0000 L CNN
-F 2 "Capacitor_SMD:C_0603_1608Metric_Pad1.05x0.95mm_HandSolder" H 1838 1500 50  0001 C CNN
-F 3 "~" H 1800 1650 50  0001 C CNN
-	1    1800 1650
-	1    0    0    1
-$EndComp
-$Comp
-L Device:D_Schottky D1
-U 1 1 5BDE4886
-P 2350 1700
-F 0 "D1" V 2350 1750 50  0000 L CNN
-F 1 "D_Schottky" V 2450 1750 50  0000 L CNN
-F 2 "Diode_SMD:D_0603_1608Metric_Pad1.05x0.95mm_HandSolder" H 2350 1700 50  0001 C CNN
-F 3 "~" H 2350 1700 50  0001 C CNN
-	1    2350 1700
-	0    1    1    0
-$EndComp
-$Comp
-L pspice:INDUCTOR L1
-U 1 1 5BDE5512
-P 2100 1500
-F 0 "L1" H 2100 1350 50  0000 C CNN
-F 1 "47uH" H 2100 1450 50  0000 C CNN
-F 2 "LightingBoard_Hardware2:ETQ-P4M470YFN_Inductor" H 2100 1500 50  0001 C CNN
-F 3 "~" H 2100 1500 50  0001 C CNN
-	1    2100 1500
-	-1   0    0    -1
-$EndComp
-$Comp
-L Device:C C3
-U 1 1 5BDE8642
-P 2900 1150
-F 0 "C3" V 2648 1150 50  0000 C CNN
-F 1 "10uF" V 2739 1150 50  0000 C CNN
-F 2 "Capacitor_SMD:C_0603_1608Metric_Pad1.05x0.95mm_HandSolder" H 2938 1000 50  0001 C CNN
-F 3 "~" H 2900 1150 50  0001 C CNN
-	1    2900 1150
-	0    1    1    0
-$EndComp
-$Comp
-L power:+5V #PWR0101
-U 1 1 5C04B7FB
-P 1750 1500
-F 0 "#PWR0101" H 1750 1350 50  0001 C CNN
-F 1 "+5V" H 1765 1673 50  0000 C CNN
-F 2 "" H 1750 1500 50  0001 C CNN
-F 3 "" H 1750 1500 50  0001 C CNN
-	1    1750 1500
-	1    0    0    -1
-$EndComp
-$Comp
-L power:GND #PWR0102
-U 1 1 5C04B898
-P 3450 1500
-F 0 "#PWR0102" H 3450 1250 50  0001 C CNN
-F 1 "GND" H 3455 1327 50  0000 C CNN
-F 2 "" H 3450 1500 50  0001 C CNN
-F 3 "" H 3450 1500 50  0001 C CNN
-	1    3450 1500
-	1    0    0    -1
-$EndComp
 Text Notes 925  900  0    197  ~ 39
 Power
@@
 L power:GND #PWR0108
 U 1 1 5C07716C
-P 1350 2100
-F 0 "#PWR0108" H 1350 1850 50  0001 C CNN
-F 1 "GND" H 1355 1927 50  0000 C CNN
-F 2 "" H 1350 2100 50  0001 C CNN
-F 3 "" H 1350 2100 50  0001 C CNN
-	1    1350 2100
+P 2350 1800
+F 0 "#PWR0108" H 2350 1550 50  0001 C CNN
+F 1 "GND" H 2355 1627 50  0000 C CNN
+F 2 "" H 2350 1800 50  0001 C CNN
+F 3 "" H 2350 1800 50  0001 C CNN
+	1    2350 1800
 	1    0    0    -1
 $EndComp
@@
 Wire Wire Line
 	4800 1900 4850 1900
-$Comp
-L MRDT_ICs:AP1059 U4
-U 1 1 5BDE0F64
-P 2700 1750
-F 0 "U4" H 3100 1700 60  0000 C CNN
-F 1 "AP1059" H 2900 2200 60  0000 C CNN
-F 2 "Package_SO:SO-8_5.3x6.2mm_P1.27mm" H 2450 1650 60  0001 C CNN
-F 3 "" H 2450 1650 60  0001 C CNN
-	1    2700 1750
-	1    0    0    -1
-$EndComp
 Wire Wire Line
 	1050 1800 1100 1800
 Wire Wire Line
 	1050 2100 1350 2100
-Wire Wire Line
-	1050 1400 2500 1400
-Wire Wire Line
-	2500 1400 2500 1150
-Wire Wire Line
-	2500 1150 2750 1150
-Connection ~ 2500 1400
-Wire Wire Line
-	3050 1150 3350 1150
-Wire Wire Line
-	3350 1150 3350 1400
-Wire Wire Line
-	3350 1400 3350 1500
-Connection ~ 3350 1400
-Connection ~ 3350 1500
-Wire Wire Line
-	3350 1500 3350 1600
-Connection ~ 3350 1600
-Wire Wire Line
-	3350 1600 3350 1700
-Wire Wire Line
-	3350 1500 3450 1500
-Wire Wire Line
-	2500 1700 2500 1850
-Wire Wire Line
-	2500 1850 3350 1850
-Wire Wire Line
-	3350 1850 3350 1700
-Connection ~ 3350 1700
-Wire Wire Line
-	2350 1500 2500 1500
-Connection ~ 2500 1850
-Wire Wire Line
-	1750 1500 1800 1500
-Connection ~ 1800 1500
-Wire Wire Line
-	1800 1500 1850 1500
-Wire Wire Line
-	1800 1800 1800 1850
-Wire Wire Line
-	1800 1850 2350 1850
-Connection ~ 2350 1850
-Wire Wire Line
-	2350 1850 2500 1850
-Wire Wire Line
-	2350 1550 2350 1500
-Connection ~ 2350 1500
-Wire Wire Line
-	2500 1600 1850 1600
-Wire Wire Line
-	1850 1600 1850 1500
-Connection ~ 1850 1500
 $Comp
 L power:+12VA #PWR?
@@
 Wire Wire Line
 	5300 3850 5750 3850
+$Comp
+L MRDT_Devices:OKI U?
+U 1 1 5C15F42F
+P 2150 1500
+F 0 "U?" H 2200 1450 60  0001 C CNN
+F 1 "OKI" H 2350 1781 60  0000 C CNN
+F 2 "" H 1950 1400 60  0001 C CNN
+F 3 "" H 1950 1400 60  0001 C CNN
+	1    2150 1500
+	1    0    0    -1
+$EndComp
+Wire Wire Line
+	1950 1400 1850 1400
+$Comp
+L power:GND #PWR?
+U 1 1 5C1613C0
+P 1350 2100
+F 0 "#PWR?" H 1350 1850 50  0001 C CNN
+F 1 "GND" H 1355 1927 50  0000 C CNN
+F 2 "" H 1350 2100 50  0001 C CNN
+F 3 "" H 1350 2100 50  0001 C CNN
+	1    1350 2100
+	1    0    0    -1
+$EndComp
+Wire Wire Line
+	2350 1700 2350 1750
+$Comp
+L power:+5V #PWR?
+U 1 1 5C1614A1
+P 2850 1400
+F 0 "#PWR?" H 2850 1250 50  0001 C CNN
+F 1 "+5V" H 2850 1550 50  0000 C CNN
+F 2 "" H 2850 1400 50  0001 C CNN
+F 3 "" H 2850 1400 50  0001 C CNN
+	1    2850 1400
+	-1   0    0    -1
+$EndComp
+Wire Wire Line
+	2750 1400 2800 1400
+$Comp
+L Device:C_Small C?
+U 1 1 5C167967
+P 2800 1550
+F 0 "C?" H 2950 1600 50  0000 L CNN
+F 1 "10uF" H 2900 1500 50  0000 L CNN
+F 2 "Capacitor_SMD:C_0603_1608Metric_Pad1.05x0.95mm_HandSolder" H 2838 1400 50  0001 C CNN
+F 3 "~" H 2800 1550 50  0001 C CNN
+	1    2800 1550
+	-1   0    0    -1
+$EndComp
+$Comp
+L Device:C_Small C?
+U 1 1 5C1679DF
+P 1850 1550
+F 0 "C?" H 2000 1600 50  0000 L CNN
+F 1 "10uF" H 1950 1500 50  0000 L CNN
+F 2 "Capacitor_SMD:C_0603_1608Metric_Pad1.05x0.95mm_HandSolder" H 1888 1400 50  0001 C CNN
+F 3 "~" H 1850 1550 50  0001 C CNN
+	1    1850 1550
+	-1   0    0    -1
+$EndComp
+Wire Wire Line
+	2800 1450 2800 1400
+Connection ~ 2800 1400
+Wire Wire Line
+	2800 1400 2850 1400
+Wire Wire Line
+	2800 1650 2800 1750
+Wire Wire Line
+	2800 1750 2350 1750
+Connection ~ 2350 1750
+Wire Wire Line
+	2350 1750 2350 1800
+Wire Wire Line
+	1850 1450 1850 1400
+Connection ~ 1850 1400
+Wire Wire Line
+	1850 1400 1050 1400
+Wire Wire Line
+	1850 1650 1850 1750
+Wire Wire Line
+	1850 1750 2350 1750
 $EndSCHEMATC

Commit message: Fixed Scematic for the nth time
Parts:
- U4: renamed from U?; footprint (none) -> MRDT_Devices:OKI_Horizontal
- gave numbers to parts that had none: 2
- renumbered Conn1 to Conn2, Conn2 to Conn3, Conn3 to Conn4
Changed lines of the file:
@@
 Headlight_V1-
 $Comp
-L MRDT_Connectors:Molex_SL_02 Conn1
+L MRDT_Connectors:Molex_SL_02 Conn2
 U 1 1 5BD0353C
 P 3100 3700
-F 0 "Conn1" H 3227 3858 60  0000 L CNN
+F 0 "Conn2" H 3227 3858 60  0000 L CNN
 F 1 "Molex_SL_02" H 3227 3752 60  0000 L CNN
 F 2 "MRDT_Connectors:MOLEX_SL_02_Horizontal" H 3100 3600 60  0001 C CNN
@@
 Headlight_V2-
 $Comp
-L MRDT_Connectors:Molex_SL_02 Conn2
+L MRDT_Connectors:Molex_SL_02 Conn3
 U 1 1 5BD053FB
 P 3100 4700
-F 0 "Conn2" H 3227 4858 60  0000 L CNN
+F 0 "Conn3" H 3227 4858 60  0000 L CNN
 F 1 "Molex_SL_02" H 3227 4752 60  0000 L CNN
 F 2 "MRDT_Connectors:MOLEX_SL_02_Horizontal" H 3100 4600 60  0001 C CNN
@@
 	8100 475  8100 5075
 $Comp
-L power:+12VA #PWR?
+L power:+12VA #PWR0101
 U 1 1 5C0C9370
 P 1400 3400
-F 0 "#PWR?" H 1400 3250 50  0001 C CNN
+F 0 "#PWR0101" H 1400 3250 50  0001 C CNN
 F 1 "+12VA" H 1415 3573 50  0000 C CNN
 F 2 "" H 1400 3400 50  0001 C CNN
@@
 	1050 2100 1350 2100
 $Comp
-L power:+12VA #PWR?
+L power:+12VA #PWR0102
 U 1 1 5C0DFFB4
 P 1350 4350
-F 0 "#PWR?" H 1350 4200 50  0001 C CNN
+F 0 "#PWR0102" H 1350 4200 50  0001 C CNN
 F 1 "+12VA" H 1365 4523 50  0000 C CNN
 F 2 "" H 1350 4350 50  0001 C CNN
@@
 	1450 4400 1450 4350
 $Comp
-L MRDT_Connectors:Molex_SL_03 Conn3
+L MRDT_Connectors:Molex_SL_03 Conn4
 U 1 1 5C05D1B6
 P 5100 4100
-F 0 "Conn3" H 5227 4308 60  0000 L CNN
+F 0 "Conn4" H 5227 4308 60  0000 L CNN
 F 1 "Molex_SL_03" H 5227 4202 60  0000 L CNN
 F 2 "MRDT_Connectors:MOLEX_SL_03_Horizontal" H 5100 4100 60  0001 C CNN
@@
 	5300 3850 5750 3850
 $Comp
-L MRDT_Devices:OKI U?
+L MRDT_Devices:OKI U4
 U 1 1 5C15F42F
 P 2150 1500
-F 0 "U?" H 2200 1450 60  0001 C CNN
+F 0 "U4" H 2200 1450 60  0001 C CNN
 F 1 "OKI" H 2350 1781 60  0000 C CNN
-F 2 "" H 1950 1400 60  0001 C CNN
+F 2 "MRDT_Devices:OKI_Horizontal" H 1950 1400 60  0001 C CNN
 F 3 "" H 1950 1400 60  0001 C CNN
 	1    2150 1500
@@
 	1950 1400 1850 1400
 $Comp
-L power:GND #PWR?
+L power:GND #PWR0115
 U 1 1 5C1613C0
 P 1350 2100
-F 0 "#PWR?" H 1350 1850 50  0001 C CNN
+F 0 "#PWR0115" H 1350 1850 50  0001 C CNN
 F 1 "GND" H 1355 1927 50  0000 C CNN
 F 2 "" H 1350 2100 50  0001 C CNN
@@
 	2350 1700 2350 1750
 $Comp
-L power:+5V #PWR?
+L power:+5V #PWR0116
 U 1 1 5C1614A1
 P 2850 1400
-F 0 "#PWR?" H 2850 1250 50  0001 C CNN
+F 0 "#PWR0116" H 2850 1250 50  0001 C CNN
 F 1 "+5V" H 2850 1550 50  0000 C CNN
 F 2 "" H 2850 1400 50  0001 C CNN
@@
 	2750 1400 2800 1400
 $Comp
-L Device:C_Small C?
+L Device:C_Small C3
 U 1 1 5C167967
 P 2800 1550
-F 0 "C?" H 2950 1600 50  0000 L CNN
+F 0 "C3" H 2950 1600 50  0000 L CNN
 F 1 "10uF" H 2900 1500 50  0000 L CNN
 F 2 "Capacitor_SMD:C_0603_1608Metric_Pad1.05x0.95mm_HandSolder" H 2838 1400 50  0001 C CNN
@@
 $EndComp
 $Comp
-L Device:C_Small C?
+L Device:C_Small C2
 U 1 1 5C1679DF
 P 1850 1550
-F 0 "C?" H 2000 1600 50  0000 L CNN
+F 0 "C2" H 2000 1600 50  0000 L CNN
 F 1 "10uF" H 1950 1500 50  0000 L CNN
 F 2 "Capacitor_SMD:C_0603_1608Metric_Pad1.05x0.95mm_HandSolder" H 1888 1400 50  0001 C CNN

Commit message: PCB Layout Finished
Parts:
- U1, U2: footprint Project Library:LDD-1500L_LED_DRIVER -> MRDT_Devices:LDD-1500L_LED_DRIVER
- U3: footprint MRDT_Shields:TM4C129E_Launchpad_X9_Bottom_SMD -> MRDT_Shields:TM4C129E_Launchpad_X9_SMD
Changed lines of the file:
@@
 F 0 "U3" H 6800 3400 60  0000 L CNN
 F 1 "TM4C129E_Launchpad" H 5900 2250 60  0000 L CNN
-F 2 "MRDT_Shields:TM4C129E_Launchpad_X9_Bottom_SMD" H 7000 2250 60  0001 C CNN
+F 2 "MRDT_Shields:TM4C129E_Launchpad_X9_SMD" H 7000 2250 60  0001 C CNN
 F 3 "" H 7000 2250 60  0001 C CNN
 	2    7000 2250
@@
 F 0 "U3" H 5700 3400 60  0000 L CNN
 F 1 "TM4C129E_Launchpad" H 6250 2950 60  0001 L CNN
-F 2 "MRDT_Shields:TM4C129E_Launchpad_X9_Bottom_SMD" H 5650 2250 60  0001 C CNN
+F 2 "MRDT_Shields:TM4C129E_Launchpad_X9_SMD" H 5650 2250 60  0001 C CNN
 F 3 "" H 5650 2250 60  0001 C CNN
 	3    5650 2250
@@
 F 0 "U3" H 5100 3400 60  0000 L CNN
 F 1 "TM4C129E_Launchpad" H 5450 2850 60  0001 L CNN
-F 2 "MRDT_Shields:TM4C129E_Launchpad_X9_Bottom_SMD" H 5050 2250 60  0001 C CNN
+F 2 "MRDT_Shields:TM4C129E_Launchpad_X9_SMD" H 5050 2250 60  0001 C CNN
 F 3 "" H 5050 2250 60  0001 C CNN
 	4    5050 2250
@@
 F 0 "U3" H 7630 3527 60  0001 C CNN
 F 1 "TM4C129E_Launchpad" H 7650 3400 60  0001 C CNN
-F 2 "MRDT_Shields:TM4C129E_Launchpad_X9_Bottom_SMD" H 7600 2250 60  0001 C CNN
+F 2 "MRDT_Shields:TM4C129E_Launchpad_X9_SMD" H 7600 2250 60  0001 C CNN
 F 3 "" H 7600 2250 60  0001 C CNN
 	1    7600 2250
@@
 F 0 "U1" H 1900 4747 60  0000 C CNN
 F 1 "LDD-1500L" H 1900 4641 60  0000 C CNN
-F 2 "Project Library:LDD-1500L_LED_DRIVER" H 1650 3950 60  0001 C CNN
+F 2 "MRDT_Devices:LDD-1500L_LED_DRIVER" H 1650 3950 60  0001 C CNN
 F 3 "" H 1650 3950 60  0001 C CNN
 	1    1650 3950
@@
 F 0 "U2" H 1900 5697 60  0000 C CNN
 F 1 "LDD-1500L" H 1900 5591 60  0000 C CNN
-F 2 "Project Library:LDD-1500L_LED_DRIVER" H 1650 4900 60  0001 C CNN
+F 2 "MRDT_Devices:LDD-1500L_LED_DRIVER" H 1650 4900 60  0001 C CNN
 F 3 "" H 1650 4900 60  0001 C CNN
 	1    1650 4900

Commit message: Rev2 Probably
Parts:
- removed R1: 470, Resistor_SMD:R_0603_1608Metric_Pad1.05x0.95mm_HandSolder, symbol Device:R
- renumbered D2 to D1, D3 to D2, D4 to D3, R2 to R1, R3 to R2, R4 to R3
Changed lines of the file:
@@
 Text GLabel 4800 1800 0    50   Output ~ 0
 Headlight_OnOff_PWM2
-$Comp
-L Device:R R1
-U 1 1 5BD09437
-P 5200 3650
-F 0 "R1" V 5100 3650 50  0000 C CNN
-F 1 "470" V 5200 3650 50  0000 C CNN
-F 2 "Resistor_SMD:R_0603_1608Metric_Pad1.05x0.95mm_HandSolder" V 5130 3650 50  0001 C CNN
-F 3 "~" H 5200 3650 50  0001 C CNN
-	1    5200 3650
-	0    1    1    0
-$EndComp
 Text Notes 925  900  0    197  ~ 39
 Power
@@
 Indicators
 $Comp
-L Device:R R2
+L Device:R R1
 U 1 1 5C07EDC4
 P 8650 2100
-F 0 "R2" H 8720 2146 50  0000 L CNN
+F 0 "R1" H 8720 2146 50  0000 L CNN
 F 1 "500" V 8650 2025 50  0000 L CNN
 F 2 "Resistor_SMD:R_0603_1608Metric_Pad1.05x0.95mm_HandSolder" V 8580 2100 50  0001 C CNN
@@
 $EndComp
 $Comp
-L Device:R R3
+L Device:R R2
 U 1 1 5C07EEA5
 P 9050 2100
-F 0 "R3" H 9120 2146 50  0000 L CNN
+F 0 "R2" H 9120 2146 50  0000 L CNN
 F 1 "500" V 9050 2025 50  0000 L CNN
 F 2 "Resistor_SMD:R_0603_1608Metric_Pad1.05x0.95mm_HandSolder" V 8980 2100 50  0001 C CNN
@@
 $EndComp
 $Comp
-L Device:R R4
+L Device:R R3
 U 1 1 5C07EF77
 P 9575 2100
-F 0 "R4" H 9645 2146 50  0000 L CNN
+F 0 "R3" H 9645 2146 50  0000 L CNN
 F 1 "500" V 9575 2025 50  0000 L CNN
 F 2 "Resistor_SMD:R_0603_1608Metric_Pad1.05x0.95mm_HandSolder" V 9505 2100 50  0001 C CNN
@@
 $EndComp
 $Comp
-L Device:LED D2
+L Device:LED D1
 U 1 1 5C07F18A
 P 8650 2450
-F 0 "D2" V 8688 2333 50  0000 R CNN
+F 0 "D1" V 8688 2333 50  0000 R CNN
 F 1 "G_LED" V 8597 2333 50  0000 R CNN
 F 2 "LED_SMD:LED_0603_1608Metric_Pad1.05x0.95mm_HandSolder" H 8650 2450 50  0001 C CNN
@@
 $EndComp
 $Comp
-L Device:LED D3
+L Device:LED D2
 U 1 1 5C07F262
 P 9050 2450
-F 0 "D3" V 9088 2333 50  0000 R CNN
+F 0 "D2" V 9088 2333 50  0000 R CNN
 F 1 "Org_LED" V 8997 2333 50  0000 R CNN
 F 2 "LED_SMD:LED_0603_1608Metric_Pad1.05x0.95mm_HandSolder" H 9050 2450 50  0001 C CNN
@@
 $EndComp
 $Comp
-L Device:LED D4
+L Device:LED D3
 U 1 1 5C07F2D6
 P 9575 2450
-F 0 "D4" V 9613 2333 50  0000 R CNN
+F 0 "D3" V 9613 2333 50  0000 R CNN
 F 1 "Org_LED" V 9522 2333 50  0000 R CNN
 F 2 "LED_SMD:LED_0603_1608Metric_Pad1.05x0.95mm_HandSolder" H 9575 2450 50  0001 C CNN
@@
 	5350 3950 5350 3650
 Wire Wire Line
-	4900 3650 5050 3650
-Wire Wire Line
 	6700 1300 6800 1300
 Wire Wire Line
@@
 Wire Wire Line
 	1850 1750 2350 1750
+Wire Wire Line
+	4900 3650 5350 3650
 $EndSCHEMATC
