File: Multimedia Board/Multimedia Board.sch (KiCad schematic (older format))
At the start: 20 parts, among them J1 SD_Card, U1 LM386, U2 LDD-1500L, U3 LDD-1500L

Commit message: setup TIVA, 3.3V, 5V, Aux sections
Parts:
- removed C1: 10uF, symbol Device:C
- removed C2: 10uF, symbol Device:CP
- removed C2: 0.05uF, symbol Device:C
- removed C3: 250uF, symbol Device:CP
- removed Conn1, Conn2: Molex_SL_02, symbol MRDT_Connectors:Molex_SL_02
- removed Conn3: Molex_SL_03, symbol MRDT_Connectors:Molex_SL_03
- removed LS1: Speaker, symbol Device:Speaker
- removed R1: 10, symbol Device:R
- removed RV1: R_POT, symbol Device:R_POT
- removed U1: LM386, symbol Amplifier_Audio:LM386
- removed U2, U3: LDD-1500L, symbol MRDT_Devices:LDD-1500L
- removed U? (x5): TM4C129Breakout, symbol MRDT_Shields:TM4C129Breakout
- added C? (x2): 1000uF, symbol Device:C
- added C?: 100uF, symbol Device:C
- added Conn? (x2): Molex_SL_02, symbol MRDT_Connectors:Molex_SL_02
- added Conn?: Molex_SL_03, symbol MRDT_Connectors:Molex_SL_03
- added Conn? (x2): AndersonPP, symbol MRDT_Connectors:AndersonPP
- added D? (x2): D_Schottky, symbol Device:D_Schottky
- added D? (x2): LED, symbol Device:LED
- added J?: AudioJack2_Ground, symbol Connector:AudioJack2_Ground
- added J? (x2): Test_Point, symbol MRDT_Connectors:Test_Point
- added L? (x2): L, symbol Device:L
- added R?: 500, symbol Device:R
- added R?: 330, symbol Device:R
- added U? (x8): TM4C129E_Launchpad, symbol MRDT_Shields:TM4C129E_Launchpad
- added U?: LDD-1500L, symbol MRDT_Devices:LDD-1500L
- added U?: LM2576SX-5, symbol MRDT_Devices:LM2576D2TR4
- added U?: LM2576SX-3.3, symbol MRDT_Devices:LM2576D2TR4
Connections:
- net labels added: +5V, 5V, AuxS, AuxT
- net labels removed: +5VA, Dout_Audio
- wire segments 94 -> 100
Other:
- moved on the sheet: C4
