File: Multimedia Board/MultimediaAndBlackBoxBoard/MultimediaAndBlackBoxBoard.kicad_pcb (KiCad board)
At the start: 2 copper layers, 37 parts, among them J1 104031-0811, U1 5V_OKI, U2 3V3_OKI, U3 BDJ2GA5WEFJ, U4 DS1307Z+, U5 4050, U6 Raspberry_Pi, Y1 32.768KHz

Commit message: deleted ugly traces, added nice pretty ones
Parts:
- moved C7 93.2 mm to (145.4, 54.4), turned to 180 degrees
- moved D3 89.9 mm to (144.3, 74.8), turned to 90 degrees
- moved R6 86.7 mm to (144.3, 71.0), turned to 90 degrees
- moved R1 73.3 mm to (174.9, 72.4)
- moved R2 12.3 mm to (149.5, 52.6), turned to 0 degrees
- moved R10 11.7 mm to (163.1, 71.0)
- moved R11 11.7 mm to (151.6, 71.0)
- moved R12 11.7 mm to (155.4, 71.0)
- moved R4 11.7 mm to (159.3, 71.0)
- moved R8 11.7 mm to (147.8, 71.0)
- moved D1 11.7 mm to (159.3, 74.8)
- moved D4 11.7 mm to (155.4, 74.8)
- moved D5 11.7 mm to (151.6, 74.8)
- moved D6 11.7 mm to (147.8, 74.8)
- moved D8 11.7 mm to (163.1, 74.8)
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Routing:
- net +12V: track 0.00 -> 22.1 mm
- net +5V: track 0.00 -> 20.1 mm
- net +3V3: track 0.00 -> 3.56 mm
- net Net-(U4-Pad1): track 0.00 -> 3.37 mm
- net Net-(U4-Pad2): track 0.00 -> 2.86 mm
- net SCL: track 0.00 -> 2.76 mm
- net Net-(R1-Pad2): track 0.00 -> 2.32 mm
- net Net-(D9-Pad2): track 0.00 -> 2.06 mm
- net Net-(D8-Pad2): track 0.00 -> 2.06 mm
- net Net-(D6-Pad2): track 0.00 -> 2.06 mm
- net Net-(D5-Pad2): track 0.00 -> 2.06 mm
- net Net-(D4-Pad2): track 0.00 -> 2.06 mm
- net Net-(D2-Pad2): track 0.00 -> 2.06 mm
- net Net-(D1-Pad2): track 0.00 -> 2.06 mm
- net Net-(D3-Pad2): track 0.00 -> 2.06 mm
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- added copper zone on B.Cu, net GND
- removed copper zone on B.Cu, net (none)

Commit message: traces redone
Routing:
- net Net-(Conn2-Pad1): track 1.27 -> 17.6 mm, vias 0 -> 1

Commit message: Finished layout
Parts:
- U1: value 5V_OKI -> OKI
- U2: value 3V3_OKI -> OKI
- moved U5 0.66 mm to (181.4, 85.6), turned to 270 degrees
Connections:
- Conn5 pad 1: GND -> (no net)
- Conn5 pad 2: (no net) -> +5VA
- U4 pad 3: Net-(Conn5-Pad+V) -> +5VA
- U4 pad 4: Net-(Conn5-PadGND) -> GND
Routing:
- net SD_RX: track 0.00 -> 78.2 mm, vias 0 -> 3
- net +3V3: track 3.56 -> 81.5 mm, vias 0 -> 5
- net +12VA: track 0.00 -> 77.1 mm, vias 0 -> 3
- net Dout_NeoPixel: track 0.00 -> 61.9 mm, vias 0 -> 2
- net SD_TX: track 0.94 -> 51.3 mm, vias 0 -> 2
- net SD_Select: track 0.00 -> 49.9 mm, vias 0 -> 2
- net +5VA: track 0.00 -> 48.9 mm, vias 0 -> 2
- net +5V: track 20.1 -> 66.9 mm, vias 0 -> 3
- net Net-(D1-Pad1): track 0.00 -> 43.2 mm, vias 0 -> 4
- net Net-(R4-Pad2): track 0.51 -> 40.8 mm, vias 0 -> 2
- net SDA: track 0.00 -> 31.4 mm, vias 0 -> 4
- net LightToggle: track 0.00 -> 28.8 mm
- net SCL: track 2.76 -> 27.0 mm
- net Net-(J1-Pad3): track 0.00 -> 13.6 mm, vias 0 -> 2
- net Net-(U5-Pad3): track 0.00 -> 13.4 mm, vias 0 -> 2
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
Commit message: Finished Board
Parts:
- removed D8: BLUE, LED_SMD:LED_0603_1608Metric_Pad1.05x0.95mm_HandSolder
- removed R10: 480, Resistor_SMD:R_0603_1608Metric_Pad1.05x0.95mm_HandSolder
- added G***: LOGO, Sigs:PricklySig, F.Cu at (134.1, 111.3)
- added G***: LOGO, Sigs:Alisa_Lazareva_21mmx9mm, F.Cu at (116.3, 114.8)
- moved D2 22.9 mm to (147.8, 74.8)
- moved R5 22.9 mm to (147.8, 71.0)
- moved D1 3.81 mm to (163.1, 74.8)
- moved D4 3.81 mm to (159.3, 74.8)
- moved D5 3.81 mm to (155.4, 74.8)
- moved D6 3.81 mm to (151.6, 74.8)
- moved R11 3.81 mm to (155.4, 71.0)
- moved R12 3.81 mm to (159.3, 71.0)
- moved R4 3.81 mm to (163.1, 71.0)
- moved R8 3.81 mm to (151.6, 71.0)
Routing:
- net SCL: track 27.0 -> 31.9 mm, vias 0 -> 2
- net SD_RX: track 78.2 -> 74.3 mm
- net Net-(D1-Pad1): track 43.2 -> 39.5 mm
- net SDA: track 31.4 -> 28.4 mm, vias 4 -> 2
- net Net-(D8-Pad2): track 2.06 -> 0.00 mm
- net SD_Select: track 49.9 -> 48.9 mm
- net Net-(R4-Pad2): track 40.8 -> 39.8 mm
- net Dout_NeoPixel: track 61.9 -> 62.1 mm, vias 2 -> 3
Other:
- board outline added: 124.5 x 79.2 mm
- board text added: "+"
- board text added: "+3V3"
- board text added: "+5V"
- board text added: "-"
- board text added: "ACT"
- board text added: "Dout NeoPixel"
- board text added: "INDICATORS"
- board text added: "Logic"
- board text added: "Multimedia, Rev1 Mars Rover Design Team Missouri S&T, 2020 Alex Wortmann, Alisa Lazareva"
- board text added: "POWER"
- board text added: "S"
- board text added: "SCL"
- board text added: "SDA"
- board text added: "SD_RX"
- board text added: "SD_Select"
- board text added: "SD_TX"
